File: Hardware/dragster schematic/dragster/dragster/dragster.kicad_sch (KiCad schematic)
At the start: 38 parts, among them U1 STM32L412KBTx, U2 MAX5033DUSA+T, U3 50SQ100, U4 MAX5033DUSA+T, U5 50SQ100

Commit message: correction
Parts:
- removed C14: 10n, symbol Device:C_Small
- removed C6: 47u, symbol Device:C_Small
- removed H1, H2, H3, H4: MountingHole, symbol Mechanical:MountingHole
- removed L3: 39n, symbol Device:L_Small
- removed R11: R_Small, symbol Device:R_Small
- removed U5: 50SQ100, 50QS100, symbol 50SQ100:50SQ100
- added C6: 47uF, symbol Device:C_Polarized_Small
- added D3: D_Schottky, symbol Device:D_Schottky
- added H1, H2, H3, H4: MountingHole_Pad, symbol Mechanical:MountingHole_Pad
- added J1, J2: Conn_01x02, symbol Connector_Generic:Conn_01x02
- C13: value 1u -> 100n
- R10: value 13500 -> 13.5k
Connections:
- net +3.3VA is gone; now on net +3.3V: U1.5 (VDDA)
- net +12V: now also C6.1, J1.2 (Pin_2)
- net +3.3V: now also C13.1, C9.1, L2.2, R9.1
- net GND: now also U1.16 (VSS), U1.32 (VSS), C6.2, D3.2 (A), H1.1, H2.1, H3.1, H4.1, J1.1 (Pin_1), J2.1 (Pin_1)
- net LX: now also D3.1 (K)
- net +7.5V: now reaches L1.2, R4.1, R5.1
- net +7.5V: now also J2.2 (Pin_2)
Other:
- moved on the sheet: C1, C10, C11, C12, C2, C3, C4, C5, C7, C8, C9, D1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

Commit message: Add files via upload
Parts:
- removed C3, C7: 47u, symbol Device:C_Small
- removed C4, C9: 33u, symbol Device:C_Small
- removed U3: 50SQ100, 50QS100, symbol 50SQ100:50SQ100
- added C3, C7: 47uF, Capacitor_SMD:C_0603_1608Metric_Pad1.08x0.95mm_HandSolder, symbol Device:C_Polarized_Small
- added C4, C9: 33uF, Capacitor_SMD:C_0603_1608Metric_Pad1.08x0.95mm_HandSolder, symbol Device:C_Polarized_Small
- added D2: D_Schottky, symbol Device:D_Schottky
- added D4: LED_Small, symbol Device:LED_Small
- added J3: Conn_02x07_Odd_Even, Connector_PinHeader_1.27mm:PinHeader_2x07_P1.27mm_Vertical_SMD, symbol Connector_Generic:Conn_02x07_Odd_Even
- added J4: Conn_01x08, symbol Connector_Generic:Conn_01x08
- added J5: Conn_01x03, symbol Connector_Generic:Conn_01x03
- added R11: 220, Resistor_SMD:R_0603_1608Metric_Pad0.98x0.95mm_HandSolder, symbol Device:R_Small
- C1, C10, C11, C12, C13, C2, C5, C6, C8: footprint (none) -> Capacitor_SMD:C_0603_1608Metric_Pad1.08x0.95mm_HandSolder
- H1, H2, H3, H4: footprint (none) -> MountingHole:MountingHole_3.2mm_M3_DIN965_Pad
- J1, J2: footprint (none) -> Connector_JST:JST_XH_B2B-XH-A_1x02_P2.50mm_Vertical
- L1, L2: value L_Small -> 220uH; footprint (none) -> Inductor_SMD:L_0805_2012Metric_Pad1.05x1.20mm_HandSolder
- R1, R2, R3, R5, R7, R8: footprint (none) -> Resistor_SMD:R_0603_1608Metric_Pad0.98x0.95mm_HandSolder
- R10: value 13.5k -> 13k; footprint (none) -> Resistor_SMD:R_0603_1608Metric_Pad0.98x0.95mm_HandSolder
- R4: value R_Small -> 100k; footprint (none) -> Resistor_SMD:R_0603_1608Metric_Pad0.98x0.95mm_HandSolder
- R6: value 13500 -> 13.5k; footprint (none) -> Resistor_SMD:R_0603_1608Metric_Pad0.98x0.95mm_HandSolder
- R9: value 68k -> 22k; footprint (none) -> Resistor_SMD:R_0603_1608Metric_Pad0.98x0.95mm_HandSolder
Connections:
- net +3.3V: now also C9.1, J3.3 (Pin_3), J4.1 (Pin_1)
- net +7.5V: now also C4.1; no longer R4.1
- net BST: now also C3.2, C7.2
- net GND: now also R4.2, C4.2, C9.2, D2.2 (A), J3.11 (Pin_11), J3.5 (Pin_5), J3.7 (Pin_7), J4.2 (Pin_2), J5.3 (Pin_3), R11.1
- net LX: now also C3.1, C7.1, D2.1 (K)
- net NRST: now also U1.8 (PA2), J3.12 (Pin_12)
- net SCL: now reaches U1.13 (PA7)
- net SCL: now also J4.3 (Pin_3)
- net Led_Status1: now reaches U1.19 (PA9)
- net Led_Status1: now also D4.2 (A)
- net SDA: now reaches U1.20 (PA10)
- net SDA: now also J4.4 (Pin_4)
- net SWDIO: now reaches U1.23 (PA13)
- net SWDIO: now also J3.4 (Pin_4)
- net SWDCK: now reaches U1.24 (PA14)
- net SWDCK: now also J3.6 (Pin_6)
- net Bouton_USR: now reaches U1.29 (PB6)
- net Bouton_USR: now also J3.10 (Pin_10)
- net at U1.30 (PB7): now also R4.1
- net USART2_RX: now reaches U1.6 (PA0)
- net USART2_RX: now also J3.13 (Pin_13)
- net USART2_TX: now reaches U1.9 (PA3)
- net USART2_TX: now also J3.14 (Pin_14)
- new net: D4.1 (K), R11.2
- no-connect marks 0 -> 25
Other:
- note added: "Accéléromètre"
- note added: "Microcontroleur STM32"
- note added: "PWM moteur"
- note added: "Régulateur à découpage 3.3V"
- note added: "Régulateur à découpage 7.5V"
- note added: "SWD Connector"
- note added: "Trous de fixations"
- moved on the sheet: C2, C5, C8, D3, J1, J2, L1, L2, R10, R2, R3, R5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

Commit message: Add files via upload
Parts:
- added J6: Conn_01x02, Connector_JST:JST_XH_B2B-XH-A_1x02_P2.50mm_Vertical, symbol Connector_Generic:Conn_01x02
- added R12: 100k, Resistor_SMD:R_0603_1608Metric_Pad0.98x0.95mm_HandSolder, symbol Device:R_Small
- added SW2: SW_Push, Button_Switch_SMD:SW_SPST_B3U-1000P, symbol Switch:SW_Push
- D1, D4: footprint (none) -> LED_SMD:LED_0603_1608Metric_Pad1.05x0.95mm_HandSolder
- J4: footprint (none) -> Connector_PinSocket_2.54mm:PinSocket_1x08_P2.54mm_Vertical
- J5: footprint (none) -> Connector_JST:JST_XH_B3B-XH-A_1x03_P2.50mm_Vertical
Connections:
- net +12V: now also J6.2 (Pin_2)
- net +3.3V: now also R12.1
- net Bouton_USR: now also R12.2, SW2.2; no longer J3.10 (Pin_10)
- net GND: now also J6.1 (Pin_1), SW2.1
- no-connect marks 25 -> 26
