File: Hardware/dragster schematic/dragster/dragster.kicad_sch (KiCad schematic)
At the start: 11 parts, among them U2 MAX5033DUSA+T, U3 STM32L412KBT6

Commit message: Add files via upload
Parts:
- removed C3: 47u, symbol Device:C_Small
- removed U3: STM32L412KBT6, LQFP-32, symbol 2023-04-11_09-29-33:STM32L412KBT6
- added C10, C11, C12, C13: 100n, Capacitor_SMD:C_0603_1608Metric_Pad1.08x0.95mm_HandSolder, symbol Device:C_Small
- added C3, C6, C7: 47uF, Capacitor_SMD:C_0603_1608Metric_Pad1.08x0.95mm_HandSolder, symbol Device:C_Polarized_Small
- added C4, C9: 33uF, Capacitor_SMD:C_0603_1608Metric_Pad1.08x0.95mm_HandSolder, symbol Device:C_Polarized_Small
- added C5, C8: 0.1u, Capacitor_SMD:C_0603_1608Metric_Pad1.08x0.95mm_HandSolder, symbol Device:C_Small
- added D2, D3: D_Schottky, Diode_SMD:D_2114_3652Metric_Pad1.85x3.75mm_HandSolder, symbol Device:D_Schottky
- added D4, D5, D6, D7: LED_Small, LED_SMD:LED_0603_1608Metric_Pad1.05x0.95mm_HandSolder, symbol Device:LED_Small
- added H1, H2, H3, H4: MountingHole_Pad, MountingHole:MountingHole_3.2mm_M3_DIN965_Pad, symbol Mechanical:MountingHole_Pad
- added J1, J2, J6: Conn_01x02, Connector_JST:JST_XH_B2B-XH-A_1x02_P2.50mm_Vertical, symbol Connector_Generic:Conn_01x02
- added J3: Conn_02x07_Odd_Even, Connector_PinHeader_1.27mm:PinHeader_2x07_P1.27mm_Vertical_SMD, symbol Connector_Generic:Conn_02x07_Odd_Even
- added J4: Conn_01x08, Connector_PinSocket_2.54mm:PinSocket_1x08_P2.54mm_Vertical, symbol Connector_Generic:Conn_01x08
- added J5: Conn_01x03, Connector_JST:JST_XH_B3B-XH-A_1x03_P2.50mm_Vertical, symbol Connector_Generic:Conn_01x03
- added L2: 220uH, Inductor_SMD:L_0805_2012Metric_Pad1.05x1.20mm_HandSolder, symbol Device:L_Small
- added R10: 13k, Resistor_SMD:R_0603_1608Metric_Pad0.98x0.95mm_HandSolder, symbol Device:R_Small
- added R11, R13, R14, R15: 220, Resistor_SMD:R_0603_1608Metric_Pad0.98x0.95mm_HandSolder, symbol Device:R_Small
- added R12: 100k, Resistor_SMD:R_0603_1608Metric_Pad0.98x0.95mm_HandSolder, symbol Device:R_Small
- added R5: 68k, Resistor_SMD:R_0603_1608Metric_Pad0.98x0.95mm_HandSolder, symbol Device:R_Small
- added R6: 13.5k, Resistor_SMD:R_0603_1608Metric_Pad0.98x0.95mm_HandSolder, symbol Device:R_Small
- added R7, R8: R_Small, Resistor_SMD:R_0603_1608Metric_Pad0.98x0.95mm_HandSolder, symbol Device:R_Small
- added R9: 22k, Resistor_SMD:R_0603_1608Metric_Pad0.98x0.95mm_HandSolder, symbol Device:R_Small
- added SW2: SW_Push, Button_Switch_SMD:SW_SPST_B3U-1000P, symbol Switch:SW_Push
- added U1: STM32L412KBTx, Package_QFP:LQFP-32_7x7mm_P0.8mm, symbol MCU_ST_STM32L4:STM32L412KBTx
- added U4: MAX5033DUSA+T, symbol MAX5033DUSA_T:MAX5033DUSA+T
- C1, C2: footprint (none) -> Capacitor_SMD:C_0603_1608Metric_Pad1.08x0.95mm_HandSolder
- D1: footprint (none) -> LED_SMD:LED_0603_1608Metric_Pad1.05x0.95mm_HandSolder
- L1: value L_Small -> 220uH; footprint (none) -> Inductor_SMD:L_0805_2012Metric_Pad1.05x1.20mm_HandSolder
- R1, R2, R3: footprint (none) -> Resistor_SMD:R_0603_1608Metric_Pad0.98x0.95mm_HandSolder
- R4: value R_Small -> 100k; footprint (none) -> Resistor_SMD:R_0603_1608Metric_Pad0.98x0.95mm_HandSolder
- U2: footprint SOIC127P600X175-8N -> (none)
Connections:
- net +12V: now also C6.1, J1.2 (Pin_2), J6.2 (Pin_2), R7.1, U4.7 (VIN)
- net BST: now also C3.2, C7.2, U4.1 (BST)
- net GND: now also R4.2, U2.3 (SGND), U2.6 (GND), C10.2, C11.2, C12.2, C13.2, C4.2, C5.2, C6.2, C8.2, C9.2, D2.2 (A), D3.2 (A), H1.1, H2.1, H3.1, H4.1, J1.1 (Pin_1), J2.1 (Pin_1), J3.11 (Pin_11), J3.5 (Pin_5), J3.7 (Pin_7), J4.2 (Pin_2), J5.3 (Pin_3), J6.1 (Pin_1), R10.2, R11.1, R13.2, R14.2, R15.2, R6.2, R8.2, SW2.1, U1.16 (VSS), U1.32 (VSS), U4.3 (SGND), U4.6 (GND)
- net LX: now also C3.1, D2.1 (K)
- net Led_Status: now also D5.2 (A), U1.18 (PA8); no longer D1.2 (A)
- net NRST: now also J3.12 (Pin_12), U1.4 (NRST), U1.8 (PA2)
- net VD: now reaches U2.2 (VD)
- net VD: now also C5.1
- net FB: now reaches U2.4 (FB)
- net FB: now also R10.1, R5.2, R6.1, R9.2, U4.4 (FB)
- net at R4.1: now also U1.30 (PB7); no longer L1.2
- new net: C8.1, U4.2 (VD)
- new net: R7.2, R8.1, U4.5 (ON/~OFF)
- new net: C7.1, D3.1 (K), L2.1, U4.8 (LX)
- new net: D7.1 (K), R15.1
- new net: D5.1 (K), R13.1
- new net: D6.1 (K), R14.1
- new net: D4.1 (K), R11.2
- new net +3.3V: C10.1, C11.1, C12.1, C13.1, C9.1, J3.3 (Pin_3), J4.1 (Pin_1), L2.2, R12.1, R9.1, U1.1 (VDD), U1.17 (VDD), U1.5 (VDDA)
- new net +7.5V: C4.1, J2.2 (Pin_2), L1.2, R5.1
- new net Bouton_USR: R12.2, SW2.2, U1.29 (PB6)
- new net Led_Status1: D4.2 (A), U1.19 (PA9)
- new net Led_Status2: D1.2 (A), U1.10 (PA4)
- new net Led_Status3: D6.2 (A), U1.11 (PA5)
- new net Led_Status4: D7.2 (A), U1.12 (PA6)
- new net SCL: J4.3 (Pin_3), U1.13 (PA7)
- new net SDA: J4.4 (Pin_4), U1.20 (PA10)
- new net SWDCK: J3.6 (Pin_6), U1.24 (PA14)
- new net SWDIO: J3.4 (Pin_4), U1.23 (PA13)
- new net USART2_RX: J3.13 (Pin_13), U1.6 (PA0)
- new net USART2_TX: J3.14 (Pin_14), U1.9 (PA3)
- no-connect marks 0 -> 26
Other:
- note added: "Accéléromètre"
- note added: "LED"
- note added: "Microcontroleur STM32"
- note added: "PWM moteur"
- note added: "Régulateur à découpage 3.3V"
- note added: "Régulateur à découpage 7.5V"
- note added: "SWD Connector"
- note added: "Trous de fixations"
- moved on the sheet: C1, C2, D1, L1, R1, R2, R3, U2

Commit message: Add files via upload
Parts:
- U2, U4: footprint (none) -> Package_SO:SSO-8_6.8x5.9mm_P1.27mm_Clearance7mm
Connections:
- net ESC1: now reaches U1.21 (PA11)
- net ESC1: now also J5.1 (Pin_1)
Other:
- note added: "Bouton poussoir"
Changed lines of the file:
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@@
+    (fill (type none))
+  )
+  (rectangle (start 233.68 327.66) (end 287.02 364.49)
+    (stroke (width 0) (type default))
     (fill (type none))
   )
@@
     (effects (font (size 1.27 1.27)) (justify left bottom))
   )
+  (text "Bouton poussoir" (at 236.22 331.47 0)
+    (effects (font (size 1.27 1.27)) (justify left bottom))
+  )
   (text "SWD Connector" (at 232.41 373.38 0)
     (effects (font (size 1.27 1.27)) (justify left bottom))
@@
     )
   )
+  (global_label "ESC1" (shape input) (at 524.51 334.01 180) (fields_autoplaced)
+    (effects (font (size 1.27 1.27)) (justify right))
+    (property "Intersheetrefs" "${INTERSHEET_REFS}" (at 516.7662 334.01 0)
+      (effects (font (size 1.27 1.27)) (justify right) hide)
+    )
+  )
   (global_label "GND" (shape input) (at 467.36 280.67 180) (fields_autoplaced)
     (effects (font (size 1.27 1.27)) (justify right))
@@
     )
   )
+  (global_label "ESC1" (shape input) (at 363.22 392.43 0) (fields_autoplaced)
+    (effects (font (size 1.27 1.27)) (justify left))
+    (property "Intersheetrefs" "${INTERSHEET_REFS}" (at 370.9638 392.43 0)
+      (effects (font (size 1.27 1.27)) (justify left) hide)
+    )
+  )
   (global_label "USART2_RX" (shape input) (at 363.22 364.49 0) (fields_autoplaced)
     (effects (font (size 1.27 1.27)) (justify left))
@@
       (effects (font (size 1.27 1.27)))
     )
-    (property "Footprint" "" (at 317.5 289.56 0)
+    (property "Footprint" "Package_SO:SSO-8_6.8x5.9mm_P1.27mm_Clearance7mm" (at 317.5 289.56 0)
       (effects (font (size 1.27 1.27)) (justify bottom) hide)
     )
@@
       (effects (font (size 1.27 1.27)))
     )
-    (property "Footprint" "" (at 485.14 288.29 0)
+    (property "Footprint" "Package_SO:SSO-8_6.8x5.9mm_P1.27mm_Clearance7mm" (at 485.14 288.29 0)
       (effects (font (size 1.27 1.27)) (justify bottom) hide)
     )

Commit message: Add files via upload
Parts:
- removed C2: 47u, Capacitor_SMD:C_0603_1608Metric_Pad1.08x0.95mm_HandSolder, symbol Device:C_Small
- removed C3, C7: 47uF, Capacitor_SMD:C_0603_1608Metric_Pad1.08x0.95mm_HandSolder, symbol Device:C_Polarized_Small
- removed C4: 33uF, Capacitor_SMD:C_0603_1608Metric_Pad1.08x0.95mm_HandSolder, symbol Device:C_Polarized_Small
- removed C5: 0.1u, Capacitor_SMD:C_0603_1608Metric_Pad1.08x0.95mm_HandSolder, symbol Device:C_Small
- removed J2: Conn_01x02, Connector_JST:JST_XH_B2B-XH-A_1x02_P2.50mm_Vertical, symbol Connector_Generic:Conn_01x02
- removed R12: 100k, Resistor_SMD:R_0603_1608Metric_Pad0.98x0.95mm_HandSolder, symbol Device:R_Small
- added C2: 47uF, Capacitor_SMD:C_Elec_6.3x5.4, symbol Device:C_Polarized_Small
- added C3, C4, C7: 100n, Capacitor_SMD:C_0603_1608Metric_Pad1.08x0.95mm_HandSolder, symbol Device:C_Small
- added C5: 33uF, Capacitor_SMD:C_Elec_6.3x5.4, symbol Device:C_Polarized_Small
- added J7: Conn_01x03, Connector_JST:JST_XH_B3B-XH-A_1x03_P2.50mm_Vertical, symbol Connector_Generic:Conn_01x03
- C13: value 100n -> 1u
- C6, C9: footprint Capacitor_SMD:C_0603_1608Metric_Pad1.08x0.95mm_HandSolder -> Capacitor_SMD:C_Elec_6.3x5.4
- C8: value 0.1u -> 100n
- J1, J6: footprint Connector_JST:JST_XH_B2B-XH-A_1x02_P2.50mm_Vertical -> Connector_AMASS:AMASS_XT60-M_1x02_P7.20mm_Vertical
- L1, L2: footprint Inductor_SMD:L_0805_2012Metric_Pad1.05x1.20mm_HandSolder -> Inductor_SMD:L_12x12mm_H6mm
- R2, R7: value R_Small -> 1M
- R3, R8: value R_Small -> 384k
- U2, U4: footprint Package_SO:SSO-8_6.8x5.9mm_P1.27mm_Clearance7mm -> Package_SO:SOIC-8_3.9x4.9mm_P1.27mm
Connections:
- net +12V: now also C2.1
- net +7.5V: now also C5.1, J7.2 (Pin_2)
- net BST: now also C4.2; no longer U4.1 (BST)
- net Bouton_USR: now also U1.31 (PH3); no longer U1.29 (PB6)
- net GND: now also C2.2, C3.2, C5.2, J7.1 (Pin_1)
- net Led_Status: now also U1.12 (PA6); no longer U1.18 (PA8)
- net Led_Status1: now also U1.11 (PA5); no longer U1.19 (PA9)
- net Led_Status3: now also U1.14 (PB0); no longer U1.11 (PA5)
- net Led_Status4: now also U1.15 (PB1); no longer U1.12 (PA6)
- net NRST: no longer U1.8 (PA2)
- net at D3.1 (K), L2.1, U4.8 (LX): now also C7.1
- net DATA SVM: now reaches U1.22 (PA12)
- net DATA SVM: now also J7.3 (Pin_3)
- net FB renamed FB1
- net FB1: no longer R5.2, R6.1, U2.4 (FB)
- net LX: no longer names the net of D2.1 (K), L1.1, U2.8 (LX)
- net LX: now also C4.1
- net VD: no longer names the net of U2.2 (VD)
- net VD: now also C3.1
- new net BST1: C7.2, U4.1 (BST)
- new net FB2: R5.2, R6.1, U2.4 (FB)
- no-connect marks 26 -> 22
Other:
- moved on the sheet: C1, C10, C11, C12, C13, C6, C9, D1, D3, D4, D5, D6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
